Commit message: Update files

File: my_robot/urdf/my_robot.xacro (robot description, xacro)
@@ -2,4 +2,7 @@
 <robot name="my_robot" xmlns:xacro="http://www.ros.org/wiki/xacro">
 	<xacro:include filename="$(find my_robot)/urdf/my_robot.gazebo" />
+  <gazebo reference="chassis">
+    <material>Gazebo/Wood</material>
+  </gazebo>
   <link name='chassis'>
     <pose>0 0 0.1 0 0 0</pose>
@@ -16,5 +19,5 @@
       <origin xyz="0 0 0" rpy="0 0 0"/>
       <geometry>
-        <box size=".4 .2 .1"/>
+        <box size=".4 .2 0.07"/>
       </geometry>
     </collision>
@@ -22,5 +25,5 @@
       <origin xyz="0 0 0" rpy="0 0 0"/>
       <geometry>
-        <box size=".4 .2 .1"/>
+        <box size=".6 .2 0.07"/>
       </geometry>
     </visual>
@@ -50,61 +53,135 @@
     </visual>
   </link>
-	<link name='left_wheel'>
-		<inertial>
-			<mass value="5"/>
-			<origin xyz="0.0 0 0" rpy="0 1.5757 1.5757"/>
-			<inertia
-				ixx="0.1" ixy="0" ixz="0"
-				iyy="0.1" iyz="0"
-				izz="0.1"
-			/>
-		</inertial>
-		<collision name='left_wheel_collision'>
-			<origin xyz="0 0 0" rpy="0 1.5757 1.5757"/>
-			<geometry>
-				<cylinder radius="0.1" length="0.05"/>
-			</geometry>
-		</collision>
-    <visual name='left_wheel_visual'>
-      <origin xyz="0 0 0" rpy="0 1.5757 1.5757"/>
-      <geometry>
-        <cylinder radius="0.1" length="0.05"/>
-      </geometry>
-    </visual>
-	</link>
-	<joint type="continuous" name="left_wheel_hinge">
-    <origin xyz="0 0.15 0" rpy="0 0 0"/>
-    <child link="left_wheel"/>
-    <parent link="chassis"/>
-    <axis xyz="0 1 0" rpy="0 0 0"/>
-    <limit effort="10000" velocity="1000"/>
-    <dynamics damping="1.0" friction="1.0"/>
-  </joint>
-	<link name='right_wheel'>
-		<inertial>
-			<mass value="5"/>
-			<origin xyz="0.0 0 0" rpy="0 1.5757 1.5757"/>
-			<inertia
-				ixx="0.1" ixy="0" ixz="0"
-				iyy="0.1" iyz="0"
-				izz="0.1"
-			/>
-		</inertial>
-		<collision name='right_wheel_collision'>
-			<origin xyz="0 0 0" rpy="0 1.5757 1.5757"/>
-			<geometry>
-				<cylinder radius="0.1" length="0.05"/>
-			</geometry>
-		</collision>
-    <visual name='right_wheel_visual'>
-      <origin xyz="0 0 0" rpy="0 1.5757 1.5757"/>
-      <geometry>
-        <cylinder radius="0.1" length="0.05"/>
-      </geometry>
-    </visual>
-	</link>
-  <joint type="continuous" name="right_wheel_hinge">
-    <origin xyz="0 -0.15 0" rpy="0 0 0"/>
-    <child link="right_wheel"/>
+  <gazebo reference="left_wheel_front">
+    <material>Gazebo/DarkGrey</material>
+  </gazebo>
+	<link name='left_wheel_front'>
+		<inertial>
+			<mass value="5"/>
+			<origin xyz="0.0 0 0" rpy="0 1.5757 1.5757"/>
+			<inertia
+				ixx="0.1" ixy="0" ixz="0"
+				iyy="0.1" iyz="0"
+				izz="0.1"
+			/>
+		</inertial>
+		<collision name='left_wheel_front_collision'>
+			<origin xyz="0 0 0" rpy="0 1.5757 1.5757"/>
+			<geometry>
+				<cylinder radius="0.1" length="0.05"/>
+			</geometry>
+		</collision>
+    <visual name='left_wheel_front_visual'>
+      <origin xyz="0 0 0" rpy="0 1.5757 1.5757"/>
+      <geometry>
+        <cylinder radius="0.1" length="0.05"/>
+      </geometry>
+    </visual>
+	</link>
+	<joint type="continuous" name="left_wheel_front_hinge">
+    <origin xyz=".1 0.15 0" rpy="0 0 0"/>
+    <child link="left_wheel_front"/>
+    <parent link="chassis"/>
+    <axis xyz="0 1 0" rpy="0 0 0"/>
+    <limit effort="10000" velocity="1000"/>
+    <dynamics damping="1.0" friction="1.0"/>
+  </joint>
+  <gazebo reference="left_wheel_back">
+    <material>Gazebo/DarkGrey</material>
+  </gazebo>
+  <link name='left_wheel_back'>
+		<inertial>
+			<mass value="5"/>
+			<origin xyz="0.0 0 0" rpy="0 1.5757 1.5757"/>
+			<inertia
+				ixx="0.1" ixy="0" ixz="0"
+				iyy="0.1" iyz="0"
+				izz="0.1"
+			/>
+		</inertial>
+		<collision name='left_wheel_back_collision'>
+			<origin xyz="0 0 0" rpy="0 1.5757 1.5757"/>
+			<geometry>
+				<cylinder radius="0.1" length="0.05"/>
+			</geometry>
+		</collision>
+    <visual name='left_wheel_back_visual'>
+      <origin xyz="0 0 0" rpy="0 1.5757 1.5757"/>
+      <geometry>
+        <cylinder radius="0.1" length="0.05"/>
+      </geometry>
+    </visual>
+	</link>
+	<joint type="continuous" name="left_wheel_back_hinge">
+    <origin xyz="-.2 0.15 0" rpy="0 0 0"/>
+    <child link="left_wheel_back"/>
+    <parent link="chassis"/>
+    <axis xyz="0 1 0" rpy="0 0 0"/>
+    <limit effort="10000" velocity="1000"/>
+    <dynamics damping="1.0" friction="1.0"/>
+  </joint>
+  <gazebo reference="right_wheel_front">
+    <material>Gazebo/DarkGrey</material>
+  </gazebo>
+	<link name='right_wheel_front'>
+		<inertial>
+			<mass value="5"/>
+			<origin xyz="0.0 0 0" rpy="0 1.5757 1.5757"/>
+			<inertia
+				ixx="0.1" ixy="0" ixz="0"
+				iyy="0.1" iyz="0"
+				izz="0.1"
+			/>
+		</inertial>
+		<collision name='right_wheel_front_collision'>
+			<origin xyz="0 0 0" rpy="0 1.5757 1.5757"/>
+			<geometry>
+				<cylinder radius="0.1" length="0.05"/>
+			</geometry>
+		</collision>
+    <visual name='right_wheel_front_visual'>
+      <origin xyz="0 0 0" rpy="0 1.5757 1.5757"/>
+      <geometry>
+        <cylinder radius="0.1" length="0.05"/>
+      </geometry>
+    </visual>
+	</link>
+  <joint type="continuous" name="right_wheel_front_hinge">
+    <origin xyz=".1 -0.15 0" rpy="0 0 0"/>
+    <child link="right_wheel_front"/>
+    <parent link="chassis"/>
+    <axis xyz="0 1 0" rpy="0 0 0"/>
+    <limit effort="10000" velocity="1000"/>
+    <dynamics damping="1.0" friction="1.0"/>
+  </joint>
+  <gazebo reference="right_wheel_back">
+    <material>Gazebo/DarkGrey</material>
+  </gazebo>
+  <link name='right_wheel_back'>
+		<inertial>
+			<mass value="5"/>
+			<origin xyz="0.0 0 0" rpy="0 1.5757 1.5757"/>
+			<inertia
+				ixx="0.1" ixy="0" ixz="0"
+				iyy="0.1" iyz="0"
+				izz="0.1"
+			/>
+		</inertial>
+		<collision name='right_wheel_back_collision'>
+			<origin xyz="0 0 0" rpy="0 1.5757 1.5757"/>
+			<geometry>
+				<cylinder radius="0.1" length="0.05"/>
+			</geometry>
+		</collision>
+    <visual name='right_wheel_back_visual'>
+      <origin xyz="0 0 0" rpy="0 1.5757 1.5757"/>
+      <geometry>
+        <cylinder radius="0.1" length="0.05"/>
+      </geometry>
+    </visual>
+	</link>
+  <joint type="continuous" name="right_wheel_back_hinge">
+    <origin xyz="-.2 -0.15 0" rpy="0 0 0"/>
+    <child link="right_wheel_back"/>
     <parent link="chassis"/>
     <axis xyz="0 1 0" rpy="0 0 0"/>

Commit message: Update process image

File: my_robot/urdf/my_robot.xacro (robot description, xacro)
@@ -2,4 +2,10 @@
 <robot name="my_robot" xmlns:xacro="http://www.ros.org/wiki/xacro">
 	<xacro:include filename="$(find my_robot)/urdf/my_robot.gazebo" />
+  <link name="robot_footprint"></link>
+  <joint name="robot_footprint_joint" type="fixed">
+    <origin xyz="0 0 0" rpy="0 0 0" />
+    <parent link="robot_footprint"/>
+    <child link="chassis" />
+  </joint>
   <gazebo reference="chassis">
     <material>Gazebo/Wood</material>
@@ -199,5 +205,5 @@
 			/>
 		</inertial>
-		<collision name='camera_collision'>
+		<collision name="camera_collision">
 			<origin xyz="0 0 0" rpy=" 0 0 0"/>
 			<geometry>
@@ -205,5 +211,5 @@
 			</geometry>
 		</collision>
-    <visual name='camera_visual'>
+    <visual name="camera_visual">
       <origin xyz="0 0 0" rpy=" 0 0 0"/>
       <geometry>
